File: eagle/placa_v4.sch (EAGLE design)
At the start: 33 parts, among them IC1 7805, Q1 IRF740, Y1 16MHz

Commit message: Boberinhas
git-svn-id: https://mbs-bot.googlecode.com/svn/trunk@211 3c29fe3e-da84-11de-ae71-c59d11f48c9c
Parts:
- removed C9: 100n, SparkFun:CAPPTH1
Connections:
- net +5V: now also BT.2
- net GND: now also BT.1; no longer C9.1
- net N$10: now also BT.3; no longer C9.2
Other:
- moved on the sheet: A, MOTOR_DIR-1, MOTOR_DIR-2, R3
Changed lines of the file:
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@@
 <part name="C8" library="SparkFun" deviceset="CAP" device="PTH1" value="100n"/>
 <part name="P+4" library="supply1" deviceset="+5V" device=""/>
-<part name="C9" library="SparkFun" deviceset="CAP" device="PTH1" value="100n"/>
 <part name="IC1" library="v-reg" deviceset="78XXS" device="" value="7805"/>
 <part name="P+6" library="supply1" deviceset="VCC" device=""/>
@@
 <part name="MOTOR_DIR" library="con-wago-500" deviceset="W237-102" device=""/>
 <part name="BT" library="con-lstb" deviceset="MA05-1" device=""/>
+<part name="P+9" library="supply1" deviceset="+5V" device=""/>
+<part name="GND8" library="supply1" deviceset="GND" device=""/>
 </parts>
 <sheets>
@@
 <instance part="R1" gate="G$1" x="101.6" y="35.56" rot="R270"/>
 <instance part="R2" gate="G$1" x="109.22" y="35.56" rot="R270"/>
-<instance part="R3" gate="G$1" x="-12.7" y="99.06" rot="R270"/>
+<instance part="R3" gate="G$1" x="-27.94" y="99.06" rot="R270"/>
 <instance part="Y1" gate="G$1" x="-17.78" y="76.2" rot="R90"/>
 <instance part="C1" gate="G$1" x="-25.4" y="81.28" rot="R90"/>
@@
 <instance part="C7" gate="G$1" x="121.92" y="33.02" rot="R90"/>
 <instance part="C8" gate="G$1" x="172.72" y="33.02" rot="R90"/>
-<instance part="P+4" gate="1" x="-12.7" y="109.22"/>
-<instance part="C9" gate="G$1" x="-25.4" y="91.44" rot="R90"/>
+<instance part="P+4" gate="1" x="-27.94" y="109.22"/>
 <instance part="IC1" gate="1" x="121.92" y="111.76"/>
 <instance part="P+6" gate="VCC" x="81.28" y="111.76" rot="R90"/>
@@
 <instance part="R7" gate="G$1" x="147.32" y="83.82"/>
 <instance part="GND7" gate="1" x="170.18" y="73.66"/>
-<instance part="A" gate="G$1" x="63.5" y="83.82" rot="R180"/>
+<instance part="A" gate="G$1" x="60.96" y="83.82" rot="R180"/>
 <instance part="ARMA" gate="-1" x="177.8" y="104.14" rot="R180"/>
 <instance part="ARMA" gate="-2" x="177.8" y="99.06" rot="R180"/>
@@
 <instance part="MOTOR_ESQ" gate="-1" x="109.22" y="66.04"/>
 <instance part="MOTOR_ESQ" gate="-2" x="109.22" y="60.96"/>
-<instance part="MOTOR_DIR" gate="-1" x="172.72" y="58.42" rot="R180"/>
-<instance part="MOTOR_DIR" gate="-2" x="172.72" y="53.34" rot="R180"/>
+<instance part="MOTOR_DIR" gate="-1" x="172.72" y="66.04" rot="R180"/>
+<instance part="MOTOR_DIR" gate="-2" x="172.72" y="60.96" rot="R180"/>
 <instance part="BT" gate="G$1" x="83.82" y="73.66" rot="R180"/>
+<instance part="P+9" gate="1" x="71.12" y="83.82"/>
+<instance part="GND8" gate="1" x="73.66" y="63.5"/>
 </instances>
 <busses>
@@
 <junction x="-33.02" y="35.56"/>
 <wire x1="-12.7" y1="35.56" x2="-33.02" y2="35.56" width="0.1524" layer="91"/>
-<wire x1="-33.02" y1="81.28" x2="-33.02" y2="91.44" width="0.1524" layer="91"/>
-<pinref part="C9" gate="G$1" pin="1"/>
-<wire x1="-33.02" y1="91.44" x2="-30.48" y2="91.44" width="0.1524" layer="91"/>
-<junction x="-33.02" y="81.28"/>
 <pinref part="MCU" gate="1" pin="AGND"/>
 <wire x1="-10.16" y1="40.64" x2="-12.7" y2="40.64" width="0.1524" layer="91"/>
@@
 <wire x1="170.18" y1="81.28" x2="170.18" y2="76.2" width="0.1524" layer="91"/>
 </segment>
+<segment>
+<pinref part="GND8" gate="1" pin="GND"/>
+<wire x1="73.66" y1="66.04" x2="73.66" y2="78.74" width="0.1524" layer="91"/>
+<pinref part="BT" gate="G$1" pin="1"/>
+<wire x1="73.66" y1="78.74" x2="76.2" y2="78.74" width="0.1524" layer="91"/>
+</segment>
 </net>
 <net name="N$5" class="0">
@@
 <wire x1="165.1" y1="33.02" x2="167.64" y2="33.02" width="0.1524" layer="91"/>
 <junction x="165.1" y="33.02"/>
-<wire x1="165.1" y1="40.64" x2="165.1" y2="58.42" width="0.1524" layer="91"/>
+<wire x1="165.1" y1="40.64" x2="165.1" y2="66.04" width="0.1524" layer="91"/>
 <pinref part="MOTOR_DIR" gate="-1" pin="KL"/>
-<wire x1="165.1" y1="58.42" x2="167.64" y2="58.42" width="0.1524" layer="91"/>
+<wire x1="165.1" y1="66.04" x2="167.64" y2="66.04" width="0.1524" layer="91"/>
 <junction x="165.1" y="40.64"/>
 </segment>
@@
 <junction x="177.8" y="33.02"/>
 <pinref part="MOTOR_DIR" gate="-2" pin="KL"/>
-<wire x1="167.64" y1="53.34" x2="167.64" y2="43.18" width="0.1524" layer="91"/>
+<wire x1="167.64" y1="60.96" x2="167.64" y2="43.18" width="0.1524" layer="91"/>
 <junction x="167.64" y="43.18"/>
 </segment>
@@
 <pinref part="P+4" gate="1" pin="+5V"/>
 <pinref part="R3" gate="G$1" pin="1"/>
-<wire x1="-12.7" y1="106.68" x2="-12.7" y2="104.14" width="0.1524" layer="91"/>
+<wire x1="-27.94" y1="106.68" x2="-27.94" y2="104.14" width="0.1524" layer="91"/>
 </segment>
 <segment>
@@
 <wire x1="83.82" y1="22.86" x2="83.82" y2="27.94" width="0.1524" layer="91"/>
 </segment>
+<segment>
+<pinref part="P+9" gate="1" pin="+5V"/>
+<wire x1="71.12" y1="81.28" x2="71.12" y2="76.2" width="0.1524" layer="91"/>
+<pinref part="BT" gate="G$1" pin="2"/>
+<wire x1="71.12" y1="76.2" x2="76.2" y2="76.2" width="0.1524" layer="91"/>
+</segment>
 </net>
 <net name="N$10" class="0">
 <segment>
 <pinref part="MCU" gate="1" pin="PC6(/RESET/PCINT14)"/>
-<wire x1="-10.16" y1="91.44" x2="-12.7" y2="91.44" width="0.1524" layer="91"/>
-<wire x1="-12.7" y1="91.44" x2="-17.78" y2="91.44" width="0.1524" layer="91"/>
+<wire x1="-10.16" y1="91.44" x2="-17.78" y2="91.44" width="0.1524" layer="91"/>
 <pinref part="R3" gate="G$1" pin="2"/>
-<wire x1="-17.78" y1="91.44" x2="-22.86" y2="91.44" width="0.1524" layer="91"/>
-<wire x1="-12.7" y1="91.44" x2="-12.7" y2="93.98" width="0.1524" layer="91"/>
-<junction x="-12.7" y="91.44"/>
-<wire x1="-17.78" y1="91.44" x2="-17.78" y2="101.6" width="0.1524" layer="91"/>
-<wire x1="-17.78" y1="101.6" x2="-38.1" y2="101.6" width="0.1524" layer="91"/>
-<wire x1="-38.1" y1="101.6" x2="-38.1" y2="17.78" width="0.1524" layer="91"/>
+<wire x1="-17.78" y1="91.44" x2="-27.94" y2="91.44" width="0.1524" layer="91"/>
+<wire x1="-27.94" y1="91.44" x2="-27.94" y2="93.98" width="0.1524" layer="91"/>
+<junction x="-27.94" y="91.44"/>
+<wire x1="-27.94" y1="91.44" x2="-38.1" y2="91.44" width="0.1524" layer="91"/>
+<wire x1="-38.1" y1="91.44" x2="-38.1" y2="17.78" width="0.1524" layer="91"/>
 <pinref part="JP1" gate="G$1" pin="5"/>
 <wire x1="-38.1" y1="17.78" x2="66.04" y2="17.78" width="0.1524" layer="91"/>
+<wire x1="-17.78" y1="91.44" x2="-17.78" y2="101.6" width="0.1524" layer="91"/>
+<wire x1="-17.78" y1="101.6" x2="63.5" y2="101.6" width="0.1524" layer="91"/>
+<wire x1="63.5" y1="101.6" x2="63.5" y2="73.66" width="0.1524" layer="91"/>
+<pinref part="BT" gate="G$1" pin="3"/>
+<wire x1="63.5" y1="73.66" x2="76.2" y2="73.66" width="0.1524" layer="91"/>
 <junction x="-17.78" y="91.44"/>
-<pinref part="C9" gate="G$1" pin="2"/>
 </segment>
 </net>
@@
 <pinref part="MCU" gate="1" pin="PC0(ADC0/PCINT8)"/>
 <wire x1="88.9" y1="96.52" x2="88.9" y2="93.98" width="0.1524" layer="91"/>
-<wire x1="50.8" y1="91.44" x2="58.42" y2="91.44" width="0.1524" layer="91"/>
-<wire x1="58.42" y1="91.44" x2="58.42" y2="96.52" width="0.1524" layer="91"/>
-<wire x1="58.42" y1="96.52" x2="88.9" y2="96.52" width="0.1524" layer="91"/>
+<wire x1="50.8" y1="91.44" x2="55.88" y2="91.44" width="0.1524" layer="91"/>
+<wire x1="55.88" y1="91.44" x2="55.88" y2="96.52" width="0.1524" layer="91"/>
+<wire x1="55.88" y1="96.52" x2="88.9" y2="96.52" width="0.1524" layer="91"/>
 <junction x="88.9" y="96.52"/>
 <label x="53.34" y="91.44" size="1.778" layer="95"/>
@@
 <pinref part="MCU" gate="1" pin="PC1(ADC1/PCINT9)"/>
 <pinref part="A" gate="G$1" pin="1"/>
-<wire x1="50.8" y1="88.9" x2="55.88" y2="88.9" width="0.1524" layer="91"/>
+<wire x1="50.8" y1="88.9" x2="53.34" y2="88.9" width="0.1524" layer="91"/>
 </segment>
 </net>
@@
 <pinref part="A" gate="G$1" pin="2"/>
 <pinref part="MCU" gate="1" pin="PC2(ADC2/PCINT10)"/>
-<wire x1="55.88" y1="86.36" x2="50.8" y2="86.36" width="0.1524" layer="91"/>
+<wire x1="53.34" y1="86.36" x2="50.8" y2="86.36" width="0.1524" layer="91"/>
 </segment>
 </net>
@@
 <pinref part="A" gate="G$1" pin="3"/>
 <pinref part="MCU" gate="1" pin="PC3(ADC3/PCINT11)"/>
-<wire x1="55.88" y1="83.82" x2="50.8" y2="83.82" width="0.1524" layer="91"/>
+<wire x1="53.34" y1="83.82" x2="50.8" y2="83.82" width="0.1524" layer="91"/>
 </segment>
 </net>
@@
 <pinref part="MCU" gate="1" pin="PC4(ADC4/SDA/PCINT12)"/>
 <pinref part="A" gate="G$1" pin="4"/>
-<wire x1="50.8" y1="81.28" x2="55.88" y2="81.28" width="0.1524" layer="91"/>
+<wire x1="50.8" y1="81.28" x2="53.34" y2="81.28" width="0.1524" layer="91"/>
 </segment>
 </net>
@@
 <pinref part="MCU" gate="1" pin="PC5(ADC5/SCLPCINT13)"/>
 <pinref part="A" gate="G$1" pin="5"/>
-<wire x1="50.8" y1="78.74" x2="55.88" y2="78.74" width="0.1524" layer="91"/>
-</segment>
-</net>
+<wire x1="50.8" y1="78.74" x2="53.34" y2="78.74" width="0.1524" layer="91"/>
+</segment>
+</net>
